File: IV6Clock2/IV6Clock2_base.kicad_pcb (KiCad board)
At the start: 2 copper layers, 99.1 x 45.7 mm, 42 parts, among them J1 DC005, J2 Debug, J3 Conn_01x04, J4 Conn_01x04, J5 Conn_01x04, J6 Conn_01x01, SW1 <, SW2 v, SW3 >, U1 ATmega328P-PU, U2 DS3231M, U3 TLV62568DBV, U4 AP3012KTR, U5 DS3232M

Commit message: Fixed wrong pin i/o on base board
Connections:
- U1 pad 15: LDR -> Net-(J5-Pad1)
- U1 pad 16: Net-(J5-Pad1) -> Net-(J5-Pad2)
- U1 pad 17: Net-(J5-Pad2) -> Net-(J5-Pad3)
- U1 pad 18: Net-(J5-Pad3) -> Net-(J5-Pad4)
- U1 pad 19: Net-(J5-Pad4) -> BUZ
- U1 pad 23: BUZ -> LDR
Routing:
- net LDR: track 21.1 -> 26.8 mm
- net BUZ: track 12.3 -> 8.67 mm
- net Net-(J5-Pad4): track 4.44 -> 5.50 mm
- net Net-(J5-Pad3): track 4.44 -> 5.50 mm
- net Net-(J5-Pad1): track 4.44 -> 5.50 mm
- net Net-(J5-Pad2): track 4.44 -> 5.50 mm
- removed copper zone on F.Cu, net LDR
Other:
- board text added: "IV-6 Clock [1/3] V2.1 2020-08 @SarahAlroe"
- board text removed: "IV-6 Clock [1/3] V2.0 2020-08 @SarahAlroe"
